File: hw/Humidity-measurement.kicad_sch (KiCad schematic)
At the start: 4 parts, among them U1 STM32F103C8Tx

Commit message: Connected the correct pin for ADC input
Connections:
- net at R2.2, U1.30 (PA9): now also U1.10 (PA0); no longer U1.32 (PA11)
- no-connect marks 1 -> 0
Changed lines of the file:
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@@
 (kicad_sch (version 20230121) (generator eeschema)
   (paper "A4")
-  (junction (at 139.7 80.01) (diameter 0) (color 0 0 0 0)
+  (junction (at 144.78 86.36) (diameter 0) (color 0 0 0 0)
   )
-  (no_connect (at 137.16 80.01))
   (wire (pts (xy 137.16 86.36) (xy 137.16 72.39))
     (stroke (width 0) (type default))
@@
     (stroke (width 0) (type default))
   )
-  (wire (pts (xy 139.7 80.01) (xy 134.62 80.01))
+  (wire (pts (xy 139.7 72.39) (xy 139.7 86.36))
     (stroke (width 0) (type default))
   )
-  (wire (pts (xy 139.7 80.01) (xy 139.7 72.39))
-    (stroke (width 0) (type default))
-  )
-  (wire (pts (xy 139.7 86.36) (xy 139.7 80.01))
-    (stroke (width 0) (type default))
-  )
-  (wire (pts (xy 134.62 80.01) (xy 134.62 72.39))
+  (wire (pts (xy 162.56 86.36) (xy 144.78 86.36))
     (stroke (width 0) (type default))
   )
@@
     (stroke (width 0) (type default))
   )
+  (wire (pts (xy 162.56 72.39) (xy 162.56 86.36))
+    (stroke (width 0) (type default))
+  )
